Commit message: Moving, before agging cameras

File: description/gazebo_control.xacro (robot description, xacro)
@@ -19,3 +19,19 @@
         </plugin>
     </gazebo>
+<!--    <gazebo>-->
+<!--  <plugin name="skid_steer_drive_controller" filename="libgazebo_ros_skid_steer_drive.so">-->
+<!--    <updateRate>100.0</updateRate>-->
+<!--    <robotNamespace>/</robotNamespace>-->
+<!--    <leftFrontJoint>left_front_wheel_joint</leftFrontJoint>-->
+<!--    <rightFrontJoint>right_front_wheel_joint</rightFrontJoint>-->
+<!--    <leftRearJoint>left_rear_wheel_joint</leftRearJoint>-->
+<!--    <rightRearJoint>right_rear_wheel_joint</rightRearJoint>-->
+<!--    <wheelSeparation>0.3</wheelSeparation>-->
+<!--    <wheelDiameter>0.2</wheelDiameter>-->
+<!--    <robotBaseFrame>base_link</robotBaseFrame>-->
+<!--    <torque>20</torque>-->
+<!--    <topicName>cmd_vel</topicName>-->
+<!--    <broadcastTF>false</broadcastTF>-->
+<!--  </plugin>-->
+<!--</gazebo>-->
  </robot>

File: description/inertial_macros.xacro (robot description, xacro)
@@ -30,35 +30,4 @@
         </inertial>
     </xacro:macro>
-<!--    MECANUM WHEEL MACRO-->
-    <xacro:macro name="mecanum_wheel" params="scale xyz rpy joint_name child_link">
-        <joint name="${joint_name}" type="continuous">
-        <parent link="chassis"/>
-        <child link="${child_link}"/>
-        <origin xyz="${xyz}" rpy="${rpy}" />
-        <axis xyz="0 1 0"/>
-    </joint>
-    <link name="${child_link}">
-        <visual>
-            <geometry>
-                <mesh filename="file://$(find mecanum_robot)/description/meshes/mecanum_wheel_right.STL" scale="0.0015 0.0015 0.0015"/>
-            </geometry>
-            <material name="grey"/>
-        </visual>
-        <collision>
-            <origin xyz="0 0 0" rpy="1.5708 0 0"/>
-            <geometry>
-                <cylinder radius="${scale * 51.3}" length="${scale * 49}"/>
-<!--                <cylinder radius="0.144" length="0.13"/>-->
-<!--                <cylinder radius="0.154" length="0.150"/>-->
-            </geometry>
-        </collision>
-        <xacro:inertial_cylinder mass="0.1" length="${scale * 50}" radius="${scale * 51.3}">
-            <origin xyz="0 0 0" rpy="0 0 0"/>
-        </xacro:inertial_cylinder>
-    </link>
-        <gazebo reference="${child_link}">
-        <material>Gazebo/Grey</material>
-    </gazebo>
-    </xacro:macro>
 <!--    COLORS FOR GAZEBO-->
 </robot>

File: description/mecanum.urdf.xacro (robot description, xacro)
@@ -2,4 +2,5 @@
 <robot xmlns:xacro="http://www.ros.org/wiki/xacro" name="mecanum">
     <xacro:include filename="mecanum_core.xacro"/>
-    <xacro:include filename="gazebo_control.xacro"/>
+<!--    <xacro:include filename="gazebo_control.xacro"/>-->
+    <xacro:include filename="ros2_control.xacro"/>
  </robot>

File: description/mecanum_core.xacro (robot description, xacro)
@@ -20,51 +20,82 @@
     <link name="base_link">
     </link>
-<!--    &lt;!&ndash; CHASSIS &ndash;&gt;-->
-<!--    <joint name="chassis_joint" type="fixed">-->
-<!--        <parent link="base_link"/>-->
-<!--        <child link="chassis"/>-->
-<!--        <origin xyz="0 0 0"/>-->
-<!--    </joint>-->
-<!--    <link name="chassis">-->
-<!--        <visual>-->
-<!--            <origin xyz="0 0 0.08"/>-->
-<!--            <geometry>-->
-<!--                <box size="0.4 0.24 0.08"/>-->
-<!--            </geometry>-->
-<!--            <material name="yellow"/>-->
-<!--        </visual>-->
-<!--        <collision>-->
-<!--            <origin xyz="0 0 0.08"/>-->
-<!--            <geometry>-->
-<!--                <box size="0.4 0.24 0.08"/>-->
-<!--            </geometry>-->
-<!--        </collision>-->
-<!--        <xacro:inertial_box mass="0.5" x="0.4" y="0.3" z="0.1">-->
-<!--            <origin xyz="0 0 0.15" rpy="0 0 0"/>-->
-<!--        </xacro:inertial_box>-->
-<!--    </link>-->
-<!--    <gazebo reference="chassis">-->
-<!--        <material>Gazebo/Yellow</material>-->
-<!--    </gazebo>-->
-<!--        &lt;!&ndash;    1) LEFT FRONT WHEEL&ndash;&gt;-->
-<!--    <xacro:mecanum_wheel scale="0.0015" xyz="0.125 0.1575 0.08"-->
-<!--rpy="0 1 0" joint_name="left_front_wheel_joint" child_link="left_front_wheel">-->
-<!--    </xacro:mecanum_wheel>-->
-<!--    &lt;!&ndash;    2) LEFT REAR WHEEL&ndash;&gt;-->
-<!--    <xacro:mecanum_wheel scale="0.0015" xyz="-0.125 0.1575 0.08"-->
-<!--rpy="0 1 0" joint_name="left_rear_wheel_joint" child_link="left_rear_wheel">-->
-<!--    </xacro:mecanum_wheel>-->
+    <!-- CHASSIS -->
+    <joint name="chassis_joint" type="fixed">
+        <parent link="base_link"/>
+        <child link="chassis"/>
+        <origin xyz="0 0 0"/>
+    </joint>
+    <link name="chassis">
+        <visual>
+            <origin xyz="0 0 0.1"/>
+            <geometry>
+                <box size="0.4 0.24 0.1"/>
+            </geometry>
+            <material name="yellow"/>
+        </visual>
+        <collision>
+            <origin xyz="0 0 0.1"/>
+            <geometry>
+                <box size="0.4 0.24 0.1"/>
+            </geometry>
+        </collision>
+        <xacro:inertial_box mass="0.5" x="0.4" y="0.24" z="0.1">
+            <origin xyz="0 0 0.1" rpy="0 0 0"/>
+        </xacro:inertial_box>
+    </link>
+    <gazebo reference="chassis">
+        <material>Gazebo/Yellow</material>
+    </gazebo>
+        <!--    1) LEFT FRONT WHEEL-->
+ <xacro:mecanum_wheel name="left_front" side="-1" interface="hardware_interface/EffortJointInterface" />
+  <joint name="left_front_wheel_joint" type="continuous">
+    <parent link="chassis" />
+    <child link="left_front_wheel_link" />
+    <origin rpy="0 0 1.5708"  xyz="0.125 0.15 0.1"/>
+  </joint>
+    <!--    2) LEFT REAR WHEEL-->
+ <xacro:mecanum_wheel name="left_rear" side="1" interface="hardware_interface/EffortJointInterface" />
+  <joint name="left_rear_wheel_joint" type="continuous">
+    <parent link="chassis" />
+    <child link="left_rear_wheel_link" />
+    <origin rpy="0 0 1.5708"  xyz="-0.125 0.15 0.1"/>
+  </joint>
             <!--    3) RIGHT FRONT WHEEL-->
-<!--    <xacro:mecanum_wheel scale="0.0015" xyz="0.125 -0.1575 0.08"-->
-<!--rpy="0 1 0" joint_name="right_front_wheel_joint" child_link="right_front_wheel">-->
-<!--    </xacro:mecanum_wheel>-->
-    <xacro:mecanum_wheel1 name="right" side="1" interface="hardware_interface/EffortJointInterface" />
-  <joint name="right_joint_name" type="fixed">
-    <parent link="base_link" />
-    <child link="right_wheel_link" />
+ <xacro:mecanum_wheel name="right_front" side="1" interface="hardware_interface/EffortJointInterface" />
+  <joint name="right_front_wheel_joint" type="continuous">
+    <parent link="chassis" />
+    <child link="right_front_wheel_link" />
+    <origin rpy="0 0 1.5708"  xyz="0.125 -0.15 0.1"/>
   </joint>
-<!--    &lt;!&ndash;    2) RIGHT REAR WHEEL&ndash;&gt;-->
-<!--    <xacro:mecanum_wheel scale="0.0015" xyz="-0.125 -0.1575 0.08"-->
-<!--rpy="0 1 0" joint_name="right_rear_wheel_joint" child_link="right_rear_wheel">-->
-<!--    </xacro:mecanum_wheel>-->
+    <!--    4) RIGHT REAR WHEEL-->
+ <xacro:mecanum_wheel name="right_rear" side="-1" interface="hardware_interface/EffortJointInterface" />
+  <joint name="right_rear_wheel_joint" type="continuous">
+    <parent link="chassis" />
+    <child link="right_rear_wheel_link" />
+    <origin rpy="0 0 1.5708"  xyz="-0.125 -0.15 0.1"/>
+  </joint>
+<!--    SHIT-->
+    <joint name="PERED_joint" type="fixed">
+        <parent link="chassis" />
+    <child link="PERED" />
+        <origin xyz="0.125 0 0.15"/>
+    </joint>
+       <link name="PERED">
+        <visual>
+            <origin xyz="0 0 0"/>
+            <geometry>
+                <box size="0.1 0.1 0.05"/>
+            </geometry>
+            <material name="yellow"/>
+        </visual>
+        <collision>
+            <origin xyz="0 0 0.2"/>
+            <geometry>
+                <box size="0.4 0.24 0.1"/>
+            </geometry>
+        </collision>
+    </link>
+    <gazebo reference="PERED">
+        <material>Gazebo/Yellow</material>
+    </gazebo>
  </robot>

File: description/mecanum_wheel_macro.xacro (robot description, xacro)
@@ -3,5 +3,5 @@
   <xacro:include filename="wheel.xacro" />
   <xacro:include filename="rollers.xacro"  />
-  <xacro:macro name="mecanum_wheel1" params="name side interface">
+  <xacro:macro name="mecanum_wheel" params="name side interface">
     <xacro:wheel_link name="${name}" side="${side}" />
     <xacro:rollers_link name="${name}" side="${side}" />

File: description/wheel.xacro (robot description, xacro)
@@ -28,4 +28,5 @@
       <kd value="1.0" />
       <fdir1 value="0 1 0"/>
+        <material>Gazebo/White</material>
     </gazebo>
   </xacro:macro>

Commit message: Moving, camera, depth camera, LiDAR

File: description/gazebo_control.xacro (robot description, xacro)
@@ -10,5 +10,5 @@
             <!-- Limits -->
             <max_wheel_torque>200</max_wheel_torque>
-            <max_wheel_acceleration>10.0</max_wheel_acceleration>
+            <max_whGazeeel_acceleration>10.0</max_whGazeeel_acceleration>
             <!-- Output -->
             <odometry_frame>odom</odometry_frame>

File: description/mecanum.urdf.xacro (robot description, xacro)
@@ -2,5 +2,7 @@
 <robot xmlns:xacro="http://www.ros.org/wiki/xacro" name="mecanum">
     <xacro:include filename="mecanum_core.xacro"/>
-<!--    <xacro:include filename="gazebo_control.xacro"/>-->
     <xacro:include filename="ros2_control.xacro"/>
+    <xacro:include filename="lidar.xacro"/>
+    <xacro:include filename="camera.xacro"/>
+    <xacro:include filename="depth_camera.xacro"/>
  </robot>

File: description/mecanum_core.xacro (robot description, xacro)
@@ -15,8 +15,22 @@
     <!-- CONSTANS -->
     <xacro:property name="PI" value="3.1415926535897931" />
-    <xacro:property name="wheel_radius" value="0.050" />
-    <xacro:property name="wheel_width" value="0.0505" />
+    <xacro:property name="chassis_length" value="0.4"/>
+    <xacro:property name="chassis_width" value="0.24"/>
+    <xacro:property name="chassis_height" value="0.1"/>
+    <xacro:property name="chassis_mass" value="1.0"/>
+    <xacro:property name="chassis_offset" value="0.1"/>
+    <xacro:property name="wheel_radius" value="0.3"/>
+<!--    <xacro:property name="wheel_thickness" value="0.026"/>-->
+    <xacro:property name="wheel_offset_x" value="0.125"/>
     <!-- BASE LINK -->
     <link name="base_link">
+    </link>
+    <!-- BASE_FOOTPRINT LINK -->
+    <joint name="base_footprint_joint" type="fixed">
+        <parent link="base_link"/>
+        <child link="base_footprint"/>
+        <origin xyz="0 0 0" rpy="0 0 0"/>
+    </joint>
+    <link name="base_footprint">
     </link>
     <!-- CHASSIS -->
@@ -28,18 +42,18 @@
     <link name="chassis">
         <visual>
-            <origin xyz="0 0 0.1"/>
+            <origin xyz="0 0 ${chassis_offset}"/>
             <geometry>
-                <box size="0.4 0.24 0.1"/>
+                <box size="${chassis_length} ${chassis_width} ${chassis_height}"/>
             </geometry>
             <material name="yellow"/>
         </visual>
         <collision>
-            <origin xyz="0 0 0.1"/>
+            <origin xyz="0 0 ${chassis_offset}"/>
             <geometry>
-                <box size="0.4 0.24 0.1"/>
+                <box size="${chassis_length} ${chassis_width} ${chassis_height}"/>
             </geometry>
         </collision>
-        <xacro:inertial_box mass="0.5" x="0.4" y="0.24" z="0.1">
-            <origin xyz="0 0 0.1" rpy="0 0 0"/>
+        <xacro:inertial_box mass="${chassis_mass}" x="${chassis_length}" y="${chassis_width}" z="${chassis_height}">
+            <origin xyz="0 0 ${chassis_offset}" rpy="0 0 0"/>
         </xacro:inertial_box>
     </link>
@@ -52,5 +66,5 @@
     <parent link="chassis" />
     <child link="left_front_wheel_link" />
-    <origin rpy="0 0 1.5708"  xyz="0.125 0.15 0.1"/>
+    <origin rpy="0 0 ${PI/2}"  xyz="${wheel_offset_x} ${wheel_radius/2} 0.1"/>
   </joint>
     <!--    2) LEFT REAR WHEEL-->
@@ -59,5 +73,5 @@
     <parent link="chassis" />
     <child link="left_rear_wheel_link" />
-    <origin rpy="0 0 1.5708"  xyz="-0.125 0.15 0.1"/>
+    <origin rpy="0 0 ${PI/2}"  xyz="${-wheel_offset_x} ${wheel_radius/2} ${chassis_offset}"/>
   </joint>
             <!--    3) RIGHT FRONT WHEEL-->
@@ -66,5 +80,5 @@
     <parent link="chassis" />
     <child link="right_front_wheel_link" />
-    <origin rpy="0 0 1.5708"  xyz="0.125 -0.15 0.1"/>
+    <origin rpy="0 0 ${PI/2}"  xyz="${wheel_offset_x} ${-wheel_radius/2} ${chassis_offset}"/>
   </joint>
     <!--    4) RIGHT REAR WHEEL-->
@@ -73,28 +87,34 @@
     <parent link="chassis" />
     <child link="right_rear_wheel_link" />
-    <origin rpy="0 0 1.5708"  xyz="-0.125 -0.15 0.1"/>
+    <origin rpy="0 0 ${PI/2}"  xyz="${-wheel_offset_x} ${-wheel_radius/2} ${chassis_offset}"/>
   </joint>
-<!--    SHIT-->
-    <joint name="PERED_joint" type="fixed">
+<!--    LIDAR THINGS-->
+    <xacro:property name="lidar_offset_z" value="0.15"/>
+    <xacro:property name="lidar_offset_x" value="0.1"/>
+    <xacro:property name="lidar_base_prop" value="0.1"/>
+    <joint name="lidar_joint" type="fixed">
         <parent link="chassis" />
-    <child link="PERED" />
-        <origin xyz="0.125 0 0.15"/>
+    <child link="lidar_base" />
+        <origin xyz="${lidar_offset_x} 0 ${lidar_offset_z}"/>
     </joint>
-       <link name="PERED">
+       <link name="lidar_base">
         <visual>
             <origin xyz="0 0 0"/>
             <geometry>
-                <box size="0.1 0.1 0.05"/>
+                <box size="${lidar_base_prop} ${lidar_base_prop} ${lidar_base_prop}"/>
             </geometry>
             <material name="yellow"/>
         </visual>
         <collision>
-            <origin xyz="0 0 0.2"/>
+            <origin xyz="0 0 0"/>
             <geometry>
-                <box size="0.4 0.24 0.1"/>
+                <box size="${lidar_base_prop} ${lidar_base_prop} ${lidar_base_prop}"/>
             </geometry>
         </collision>
+        <xacro:inertial_box mass="${chassis_mass/5}" x="${lidar_base_prop}" y="${lidar_base_prop}" z="${lidar_base_prop}">
+            <origin xyz="0 0 ${chassis_offset}" rpy="0 0 0"/>
+        </xacro:inertial_box>
     </link>
-    <gazebo reference="PERED">
+    <gazebo reference="lidar_base">
         <material>Gazebo/Yellow</material>
     </gazebo>

Commit message: added SLAM, mapping

File: description/gazebo_control.xacro (robot description, xacro)
@@ -19,19 +19,3 @@
         </plugin>
     </gazebo>
-<!--    <gazebo>-->
-<!--  <plugin name="skid_steer_drive_controller" filename="libgazebo_ros_skid_steer_drive.so">-->
-<!--    <updateRate>100.0</updateRate>-->
-<!--    <robotNamespace>/</robotNamespace>-->
-<!--    <leftFrontJoint>left_front_wheel_joint</leftFrontJoint>-->
-<!--    <rightFrontJoint>right_front_wheel_joint</rightFrontJoint>-->
-<!--    <leftRearJoint>left_rear_wheel_joint</leftRearJoint>-->
-<!--    <rightRearJoint>right_rear_wheel_joint</rightRearJoint>-->
-<!--    <wheelSeparation>0.3</wheelSeparation>-->
-<!--    <wheelDiameter>0.2</wheelDiameter>-->
-<!--    <robotBaseFrame>base_link</robotBaseFrame>-->
-<!--    <torque>20</torque>-->
-<!--    <topicName>cmd_vel</topicName>-->
-<!--    <broadcastTF>false</broadcastTF>-->
-<!--  </plugin>-->
-<!--</gazebo>-->
  </robot>

File: description/mecanum_core.xacro (robot description, xacro)
@@ -119,3 +119,34 @@
         <material>Gazebo/Yellow</material>
     </gazebo>
+<!--    Odometry publishing-->
+     <gazebo>
+        <plugin name="libgazebo_ros_p3d" filename="libgazebo_ros_p3d.so">
+            <frame_name>map</frame_name>
+            <body_name>base_link</body_name>
+            <update_rate>30.0</update_rate>
+            <gaussian_noise>0.01</gaussian_noise>
+        </plugin>
+      </gazebo>
  </robot>
+<!--    <gazebo>-->
+<!--      <plugin name="gazebo_ros_mecanum_diff_drive" filename="libgazebo_ros_mecanum_diff_drive.so">-->
+<!--        <commandTopic>cmd_vel</commandTopic>-->
+<!--        <odometryTopic>odom</odometryTopic>-->
+<!--        <odometryFrame>odom</odometryFrame>-->
+<!--        <robotBaseFrame>base_link</robotBaseFrame>-->
+<!--        <LeftRear>left_rear_wheel_joint</LeftRear>-->
+<!--        <LeftFront>left_front_wheel_joint</LeftFront>-->
+<!--        <RightFront>right_front_wheel_joint</RightFront>-->
+<!--        <RightRear>right_rear_wheel_joint</RightRear>-->
+<!--        <odometryRate>20</odometryRate>-->
+<!--        <publishWheelTF>true</publishWheelTF>-->
+<!--        <publishWheelJointState>true</publishWheelJointState>-->
+<!--        <WheelTorque>1</WheelTorque>-->
+<!--        <WheelSeparationW>0.5</WheelSeparationW>-->
+<!--        <WheelSeparationL>0.6</WheelSeparationL>-->
+<!--        <wheelAccel>5</wheelAccel>-->
+<!--        <wheelDiameter>0.13</wheelDiameter>-->
+<!--        <publishOdom>true</publishOdom>-->
+<!--        <isRollerModel>true</isRollerModel>-->
+<!--      </plugin>-->
+<!--</gazebo>-->

File: description/ros2_control.xacro (robot description, xacro)
@@ -51,29 +51,3 @@
       </plugin>
     </gazebo>
-<!--    <ros2_control name="GazeboSystem" type="system">-->
-<!--        <hardware>-->
-<!--            <plugin>gazebo_ros2_control/GazeboSystem</plugin>-->
-<!--        </hardware>-->
-<!--        <joint name="left_rear_wheel_joint">-->
-<!--            <command_interface name="velocity">-->
-<!--                <param name="min">-10</param>-->
-<!--                <param name="max">10</param>-->
-<!--            </command_interface>-->
-<!--            <state_interface name="velocity"/>-->
-<!--            <state_interface name="pisition"/>-->
-<!--        </joint>-->
-<!--        <joint name="left_rear_wheel_joint">-->
-<!--            <command_interface name="velocity">-->
-<!--                <param name="min">-10</param>-->
-<!--                <param name="max">10</param>-->
-<!--            </command_interface>-->
-<!--            <state_interface name="velocity"/>-->
-<!--            <state_interface name="pisition"/>-->
-<!--        </joint>-->
-<!--    </ros2_control>-->
-<!--    <gazebo>-->
-<!--        <plugin name="gazebo_ros2_control" filename="libgazebo_ros2_control.so">-->
-<!--            <parameters>$(find mecanum_robot)/config/controller_ros2.yaml</parameters>-->
-<!--        </plugin>-->
-<!--    </gazebo>-->
  </robot>
